File: audio_interface.kicad_pcb (KiCad board)
At the start: 2 copper layers, 36 x 14 mm, 27 parts, among them IC1 ATMEGA16U2, P1 USB_A, P2 EAR, P3 MIC, P5 AVR-ISP, SW1 SW_PUSH, U1 7400, Y1 CSTCE16M0V53MU

Commit message: update
Parts:
- removed D2: PWR, LEDs:LED_0805
- removed P5: AVR-ISP, Pin_Headers:Pin_Header_Straight_2x03
- removed R11: 470, Resistors_SMD:R_0603_HandSoldering
- removed U1: 7400, Housings_SOIC:SOIC-14_3.9x8.7mm_Pitch1.27mm
- added IC2: SN74LVC1G00, TO_SOT_Packages_SMD:SOT-23-5, F.Cu at (157.5, 110.5)
- added IC3: SN74LVC1G00, TO_SOT_Packages_SMD:SOT-23-5, F.Cu at (163.2, 109.9)
- added P4: EAR, Pin_Headers:Pin_Header_Straight_1x02, F.Cu at (184.8, 109.2)
- P2: value EAR -> AVR-ISP; footprint Pin_Headers:Pin_Header_Straight_1x02 -> KaiBader:Pin_Header_SMD_2x03; moved to B.Cu
- R1: value 22 -> 470
- R10: value 470 -> 270
- R3: value 18k -> 22
- R5: value 1M -> 18k
- R6: value 10k -> 1M
- R7: value 270 -> 10k
- R8: value 100k -> 270
- R9: value 270 -> 100k
- moved R8 80.3 mm to (167.6, 81.3)
- moved C5 68.7 mm to (176.5, 74.3)
- moved R5 60.9 mm to (158.1, 76.2)
- moved C4 58.0 mm to (163.8, 76.2)
- moved P3 54.6 mm to (182.9, 78.7), turned to 90 degrees
- moved R10 53.7 mm to (175.3, 83.8)
- moved R7 51.2 mm to (170.8, 75.6)
- moved R9 51.2 mm to (170.2, 109.9)
- moved R4 50.3 mm to (104.8, 81.9)
- moved SW1 50.2 mm to (114.3, 79.4)
- moved C6 48.6 mm to (177.2, 109.9)
- moved C1 47.2 mm to (117.5, 89.5)
- moved R6 46.6 mm to (163.2, 116.8)
- moved C3 43.3 mm to (160.7, 81.9)
- moved D1 39.1 mm to (130.2, 113.7)
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Connections:
- IC1 pad 19: (no net) -> PB5
- IC1 pad 21: (no net) -> PD0
- IC1 pad 6: PD0 -> (no net)
- P2 pad 1: Net-(C6-Pad1) -> MISO
- P2 pad 2: GND -> ~RESET
- R1 pad 1: Net-(IC1-Pad29) -> Net-(D1-Pad2)
- R1 pad 2: Net-(P1-Pad3) -> PB4
- R10 pad 1: Net-(D1-Pad2) -> GND
- R10 pad 2: PB4 -> Net-(C5-Pad1)
- R2 pad 1: Net-(IC1-Pad30) -> Net-(IC1-Pad29)
- R2 pad 2: Net-(P1-Pad2) -> Net-(P1-Pad3)
- R3 pad 1: Net-(C3-Pad2) -> Net-(IC1-Pad30)
- R3 pad 2: PD0 -> Net-(P1-Pad2)
- R5 pad 1: Net-(R5-Pad1) -> Net-(C3-Pad2)
- R5 pad 2: Net-(R5-Pad2) -> PD0
- R6 pad 1: Net-(C5-Pad2) -> PB5
- R6 pad 2: Net-(C4-Pad1) -> Net-(IC2-Pad1)
- R7 pad 1: GND -> Net-(C5-Pad2)
- R7 pad 2: Net-(C5-Pad2) -> Net-(C4-Pad1)
- R8 pad 1: Net-(C6-Pad2) -> GND
- R8 pad 2: Net-(R5-Pad1) -> Net-(C5-Pad2)
- R9 pad 1: GND -> Net-(C6-Pad2)
- R9 pad 2: Net-(C5-Pad1) -> PB5

Commit message: update
Parts:
- SW1: footprint Buttons_Switches_SMD:SW_SPST_EVPBF -> Buttons_Switches_SMD:SW_SPST_FSMSM
- moved R8 54.9 mm to (114.9, 96.5)
- moved C5 54.6 mm to (125.1, 92.7), turned to 180 degrees
- moved R7 53.7 mm to (120.7, 94.6)
- moved P3 52.2 mm to (132.7, 93.3), turned to 270 degrees
- moved P4 51.6 mm to (133.3, 104.8), turned to 270 degrees
- moved R10 51.3 mm to (125.1, 94.6)
- moved C3 47.5 mm to (114.9, 94.6)
- moved C4 46.2 mm to (120.7, 92.7), turned to 180 degrees
- moved R5 46.2 mm to (114.9, 92.7), turned to 180 degrees
- moved C6 46.2 mm to (132.1, 99.7), turned to 270 degrees
- moved R9 41.3 mm to (130.2, 99.7), turned to 90 degrees
- moved IC3 40.7 mm to (123.8, 99.7), turned to 270 degrees
- moved IC2 39.0 mm to (120.0, 99.7), turned to 270 degrees
- moved R6 38.9 mm to (128.3, 99.7), turned to 270 degrees
- moved P2 23.5 mm to (120.0, 122.6)
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
Commit message: update
Parts:
- removed C6: 0.047uF, Capacitors_SMD:C_0603_HandSoldering
- removed IC2, IC3: SN74LVC1G00, TO_SOT_Packages_SMD:SOT-23-5
- removed the R6 at (128.3, 99.7)
- added D2: LED, LEDs:LED-3MM, F.Cu at (125.1, 102.9)
- added Q1, Q2: BC849, TO_SOT_Packages_SMD:SOT-23, F.Cu at (119.5, 115.1)
- added R1: 470, Resistors_SMD:R_0603_HandSoldering, F.Cu at (119.5, 115.1)
- added R11: R, Resistors_SMD:R_0603_HandSoldering, F.Cu at (119.5, 115.1)
- C3: value 0.01uF -> 100nF
- C4: value 0.047uF -> 10uF
- D1: footprint LEDs:LED_0805 -> LEDs:LED-3MM
- P3: value MIC -> OUT
- R10, R8: value 270 -> R
- R6: renamed from R5; value 18k -> 1.8k
- R7: value 10k -> R
- R9: value 100k -> R
- moved C5 23.0 mm to (119.5, 115.1), turned to 0 degrees
- moved R10 21.2 mm to (119.5, 115.1)
- moved R7 20.5 mm to (119.5, 115.1)
- moved R8 19.1 mm to (119.5, 115.1)
- moved R9 18.7 mm to (119.5, 115.1), turned to 0 degrees
- moved P4 17.2 mm to (119.5, 115.1), turned to 0 degrees
- moved D1 13.4 mm to (119.5, 115.1), turned to 0 degrees
- renumbered R1 to R2, R2 to R3, R3 to R4, R4 to R5
Connections:
- C1 pad 1: ~RESET -> +5V
- IC1 pad 31: ~RESET -> +5V
- IC1 pad 32: ~RESET -> +5V
- IC1 pad 4: ~RESET -> +5V
- P1 pad 1: ~RESET -> +5V
- P2 pad 2: ~RESET -> +5V
- P3 pad 1: Net-(C5-Pad1) -> Net-(C4-Pad1)
- P4 pad 1: Net-(C6-Pad1) -> Net-(C5-Pad2)
- R10 pad 1: GND -> Net-(Q2-Pad3)
- R2 pad 1: Net-(D1-Pad2) -> Net-(D2-Pad2)
- R2 pad 2: PB4 -> PB5
- R5 pad 2: ~RESET -> +5V
- R7 pad 1: Net-(C5-Pad2) -> PC7
- R7 pad 2: Net-(C4-Pad1) -> +5V
- R8 pad 1: GND -> Net-(Q1-Pad1)
- R8 pad 2: Net-(C5-Pad2) -> Net-(Q2-Pad3)
- R9 pad 1: Net-(C6-Pad2) -> Net-(Q2-Pad3)
- R9 pad 2: PB5 -> +5V

Commit message: update
Parts:
- removed D2: LED, LEDs:LED-3MM
- removed R2: 470, Resistors_SMD:R_0603_HandSoldering
- moved C1 44.3 mm to (114.1, 131.7)
- moved R6 40.8 mm to (124.4, 132.4)
- moved C3 38.0 mm to (119.6, 132.4)
- moved Y1 37.6 mm to (132.7, 127.4)
- moved R3 35.7 mm to (143.1, 111.0)
- moved R4 34.9 mm to (130.0, 123.5)
- moved C4 34.1 mm to (125.7, 126.5)
- moved P3 33.4 mm to (112.7, 120.1), turned to 0 degrees
- moved C2 33.3 mm to (132.6, 117.6)
- moved R5 32.9 mm to (127.7, 118.2)
- moved SW1 32.4 mm to (116.8, 111.7)
- moved C5 23.8 mm to (143.2, 116.9)
- moved R1 21.2 mm to (138.9, 123.5)
- moved P2 20.4 mm to (101.1, 130.2)
- moved P4 19.8 mm to (109.1, 131.9)
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Connections:
- IC1 pad 19: PB5 -> (no net)

Commit message: update
Parts:
- P2: moved to F.Cu
- moved P2 63.4 mm to (125.7, 71.8), turned to 0 degrees
- moved P4 63.0 mm to (157.5, 91.4), turned to 90 degrees
- moved P3 51.2 mm to (157.5, 95.2), turned to 90 degrees
- moved R9 49.2 mm to (152.4, 88.3)
- moved C3 47.2 mm to (152.4, 98.4)
- moved R6 45.5 mm to (152.4, 96.5)
- moved R10 44.5 mm to (148.0, 94.6)
- moved C1 44.3 mm to (134.0, 92.1), turned to 90 degrees
- moved R11 41.8 mm to (156.8, 88.3), turned to 180 degrees
- moved C4 41.5 mm to (156.2, 98.4)
- moved R8 41.0 mm to (145.4, 91.4), turned to 270 degrees
- moved Y1 40.4 mm to (132.1, 87.0)
- moved R4 39.4 mm to (135.3, 84.5)
- moved IC1 34.7 mm to (138.4, 89.5)
- moved P1 34.0 mm to (131.4, 89.4)
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
Commit message: update
Parts:
- P2: moved to B.Cu
- moved P2 14.2 mm to (139.3, 75.9), turned to 90 degrees
- moved D1 14.0 mm to (135.3, 98.6), turned to 90 degrees
- moved R3 10.1 mm to (133.9, 92.7), turned to 270 degrees
- moved Y1 10.1 mm to (137.0, 95.8), turned to 0 degrees
- moved R7 6.10 mm to (154.1, 88.5)
- moved R10 5.99 mm to (153.9, 94.1)
- moved R5 5.80 mm to (142.5, 94.0), turned to 180 degrees
- moved SW1 4.57 mm to (143.6, 97.0)
- moved R4 4.42 mm to (133.9, 88.6), turned to 270 degrees
- moved C5 4.33 mm to (155.2, 91.3), turned to 90 degrees
- moved Q1 4.04 mm to (150.2, 87.8), turned to 270 degrees
- moved R8 4.02 mm to (147.7, 88.1)
- moved C1 3.69 mm to (135.6, 88.8)
- moved R9 3.35 mm to (155.4, 86.9)
- moved C3 3.09 mm to (155.4, 98.9)
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
Commit message: update
Parts:
- added ?: AK-S-27 Case, KaiBader:AK-S-27_Case, F.Cu at (127.0, 121.9)
- moved R3 24.8 mm to (134.6, 117.5)
- moved R4 23.2 mm to (135.9, 111.8), turned to 180 degrees
- moved SW1 22.6 mm to (146.7, 119.4)
- moved P4 22.5 mm to (156.8, 113.7)
- moved D1 22.4 mm to (139.1, 120.7)
- moved C5 22.4 mm to (153.7, 113.7)
- moved C2 22.4 mm to (136.5, 114.9)
- moved Q2 22.3 mm to (151.1, 113.7)
- moved C4 22.2 mm to (159.0, 119.5)
- moved P2 22.2 mm to (140.3, 98.2)
- moved P3 22.2 mm to (156.8, 116.8)
- moved R6 22.2 mm to (155.1, 119.5)
- moved R9 22.2 mm to (156.5, 109.1)
- moved C3 22.2 mm to (156.5, 121.2)
- moved P1 22.2 mm to (132.5, 111.6)
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Other:
- outline, holes or cut-outs redrawn

Commit message: update
Parts:
- SW1: footprint Buttons_Switches_SMD:SW_SPST_FSMSM -> Buttons_Switches_SMD:SW_SPST_EVQPE1
- moved ? 27.3 mm to (127.6, 149.2)
- moved R3 27.1 mm to (135.3, 144.5)
- moved SW1 27.1 mm to (147.3, 146.4)
- moved Y1 27.1 mm to (141.6, 144.5)
- moved C1 27.1 mm to (139.1, 137.5)
- moved C3 27.1 mm to (157.1, 148.2)
- moved C5 27.1 mm to (154.3, 140.7)
- moved IC1 27.1 mm to (142.9, 138.8)
- moved P1 27.1 mm to (133.1, 138.7)
- moved P4 27.1 mm to (157.5, 140.7)
- moved Q2 27.1 mm to (151.8, 140.7)
- moved R1 27.1 mm to (147.3, 137.5)
- moved R10 27.1 mm to (153.0, 143.3)
- moved R4 27.1 mm to (136.5, 138.8)
- moved R9 27.1 mm to (157.1, 136.1)
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Changed lines of the file:
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@@
-(kicad_pcb (version 4) (host pcbnew 0.201603250401+6648~43~ubuntu15.10.1-product)
+(kicad_pcb (version 4) (host pcbnew 0.201603270401+6651~43~ubuntu15.10.1-product)
   (general
     (links 53)
     (no_connects 53)
-    (area 119.035999 93.645999 163.402001 124.1705)
+    (area 119.670999 120.696999 163.886018 151.2015)
     (thickness 1.6)
     (drawings 0)
@@
   )
   (module Capacitors_SMD:C_0603_HandSoldering (layer F.Cu)
-    (at 138.43 110.49 90)
+    (at 139.065 137.541 90)
     (descr "Capacitor SMD 0603, hand soldering")
     (tags "capacitor 0603")
@@
   )
   (module Capacitors_SMD:C_0603_HandSoldering (layer F.Cu)
-    (at 136.525 114.935 90)
+    (at 137.16 141.986 90)
     (descr "Capacitor SMD 0603, hand soldering")
     (tags "capacitor 0603")
@@
   )
   (module Capacitors_SMD:C_0603_HandSoldering (layer F.Cu)
-    (at 156.464 121.158)
+    (at 157.099 148.209)
     (descr "Capacitor SMD 0603, hand soldering")
     (tags "capacitor 0603")
@@
   )
   (module Capacitors_SMD:C_0603_HandSoldering (layer F.Cu)
-    (at 159.004 119.507 180)
+    (at 159.639 146.558 180)
     (descr "Capacitor SMD 0603, hand soldering")
     (tags "capacitor 0603")
@@
   )
   (module Capacitors_SMD:C_0603_HandSoldering (layer F.Cu)
-    (at 153.67 113.665 90)
+    (at 154.305 140.716 90)
     (descr "Capacitor SMD 0603, hand soldering")
     (tags "capacitor 0603")
@@
   )
   (module LEDs:LED-3MM (layer F.Cu)
-    (at 139.065 120.65 90)
+    (at 139.7 147.701 90)
     (descr "LED 3mm round vertical")
     (tags "LED  3mm round vertical")
@@
   )
   (module Housings_DFN_QFN:QFN-32-1EP_5x5mm_Pitch0.5mm (layer F.Cu)
-    (at 142.24 111.76 90)
+    (at 142.875 138.811 90)
     (descr "UH Package; 32-Lead Plastic QFN (5mm x 5mm); (see Linear Technology QFN_32_05-08-1693.pdf)")
     (tags "QFN 0.5")
@@
   )
   (module Connect:USB_A (layer F.Cu)
-    (at 132.461 111.633 270)
+    (at 133.096 138.684 270)
     (descr "USB A connector")
     (tags "USB USB_A")
@@
   )
   (module KaiBader:Pin_Header_SMD_2x03 (layer B.Cu)
-    (at 140.335 98.171 90)
+    (at 140.97 125.222 90)
     (descr "Through hole pin header")
     (tags "pin header")
@@
   )
   (module Pin_Headers:Pin_Header_Straight_1x02 (layer F.Cu)
-    (at 156.845 116.84 90)
+    (at 157.48 143.891 90)
     (descr "Through hole pin header")
     (tags "pin header")
@@
   )
   (module Pin_Headers:Pin_Header_Straight_1x02 (layer F.Cu)
-    (at 156.845 113.665 90)
+    (at 157.48 140.716 90)
     (descr "Through hole pin header")
     (tags "pin header")
@@
   )
   (module TO_SOT_Packages_SMD:SOT-23 (layer F.Cu)
-    (at 151.257 109.982 270)
+    (at 151.892 137.033 270)
     (descr "SOT-23, Standard")
     (tags SOT-23)
@@
   )
   (module TO_SOT_Packages_SMD:SOT-23 (layer F.Cu)
-    (at 151.13 113.665 90)
+    (at 151.765 140.716 90)
     (descr "SOT-23, Standard")
     (tags SOT-23)
@@
   )
   (module Resistors_SMD:R_0603_HandSoldering (layer F.Cu)
-    (at 146.685 110.49 90)
+    (at 147.32 137.541 90)
     (descr "Resistor SMD 0603, hand soldering")
     (tags "resistor 0603")
@@
   )
   (module Resistors_SMD:R_0603_HandSoldering (layer F.Cu)
-    (at 134.62 117.475 270)
+    (at 135.255 144.526 270)
     (descr "Resistor SMD 0603, hand soldering")
     (tags "resistor 0603")
@@
   )
   (module Resistors_SMD:R_0603_HandSoldering (layer F.Cu)
-    (at 135.89 111.76 180)
+    (at 136.525 138.811 180)
     (descr "Resistor SMD 0603, hand soldering")
     (tags "resistor 0603")
@@
   )
   (module Resistors_SMD:R_0603_HandSoldering (layer F.Cu)
-    (at 146.685 114.935 270)
+    (at 147.32 141.986 270)
     (descr "Resistor SMD 0603, hand soldering")
     (tags "resistor 0603")
@@
   )
   (module Resistors_SMD:R_0603_HandSoldering (layer F.Cu)
-    (at 155.067 119.507 180)
+    (at 155.702 146.558 180)
     (descr "Resistor SMD 0603, hand soldering")
     (tags "resistor 0603")
@@
   )
   (module Resistors_SMD:R_0603_HandSoldering (layer F.Cu)
-    (at 155.067 110.744)
+    (at 155.702 137.795)
     (descr "Resistor SMD 0603, hand soldering")
     (tags "resistor 0603")
@@
   )
   (module Resistors_SMD:R_0603_HandSoldering (layer F.Cu)
-    (at 148.717 110.363 270)
+    (at 149.352 137.414 270)
     (descr "Resistor SMD 0603, hand soldering")
     (tags "resistor 0603")
@@
   )
   (module Resistors_SMD:R_0603_HandSoldering (layer F.Cu)
-    (at 156.464 109.093)
+    (at 157.099 136.144)
     (descr "Resistor SMD 0603, hand soldering")
     (tags "resistor 0603")
@@
   )
   (module Resistors_SMD:R_0603_HandSoldering (layer F.Cu)
-    (at 152.4 116.205)
+    (at 153.035 143.256)
     (descr "Resistor SMD 0603, hand soldering")
     (tags "resistor 0603")
@@
   )
   (module Resistors_SMD:R_0603_HandSoldering (layer F.Cu)
-    (at 159.131 110.744 180)
+    (at 159.766 137.795 180)
     (descr "Resistor SMD 0603, hand soldering")
     (tags "resistor 0603")
@@
     )
   )
-  (module Buttons_Switches_SMD:SW_SPST_FSMSM (layer F.Cu)
-    (at 146.685 119.38)
-    (descr http://www.te.com/commerce/DocumentDelivery/DDEController?Action=srchrtrv&DocNm=1437566-3&DocType=Customer+Drawing&DocLang=English)
-    (tags "SPST button tactile switch")
-    (attr smd)
-    (fp_text reference SW1 (at 0.01011 -2.60022) (layer F.SilkS)
-      (effects (font (size 1 1) (thickness 0.15)))
-    )
-    (fp_text value SW_PUSH (at 0.01011 -0.00022) (layer F.Fab)
-      (effects (font (size 1 1) (thickness 0.15)))
-    )
-    (fp_line (start -1.23989 -0.55022) (end 1.26011 -0.55022) (layer F.SilkS) (width 0.15))
-    (fp_line (start 1.26011 -0.55022) (end 1.26011 0.54978) (layer F.SilkS) (width 0.15))
-    (fp_line (start 1.26011 0.54978) (end -1.23989 0.54978) (layer F.SilkS) (width 0.15))
-    (fp_line (start -1.23989 0.54978) (end -1.23989 -0.55022) (layer F.SilkS) (width 0.15))
-    (fp_line (start -1.48989 0.79978) (end 1.51011 0.79978) (layer F.SilkS) (width 0.15))
-    (fp_line (start -1.48989 -0.80022) (end 1.51011 -0.80022) (layer F.SilkS) (width 0.15))
-    (fp_line (start 1.51011 -0.80022) (end 1.51011 0.79978) (layer F.SilkS) (width 0.15))
-    (fp_line (start -1.48989 -0.80022) (end -1.48989 0.79978) (layer F.SilkS) (width 0.15))
-    (fp_line (start -5.95 2) (end 5.95 2) (layer F.CrtYd) (width 0.05))
-    (fp_line (start 5.95 -2) (end 5.95 2) (layer F.CrtYd) (width 0.05))
-    (fp_line (start -2.98989 1.74978) (end 3.01011 1.74978) (layer F.SilkS) (width 0.15))
-    (fp_line (start -2.98989 -1.75022) (end 3.01011 -1.75022) (layer F.SilkS) (width 0.15))
-    (fp_line (start -2.98989 -1.75022) (end -2.98989 1.74978) (layer F.SilkS) (width 0.15))
-    (fp_line (start 3.01011 -1.75022) (end 3.01011 1.74978) (layer F.SilkS) (width 0.15))
-    (fp_line (start -5.95 -2) (end -5.95 2) (layer F.CrtYd) (width 0.05))
-    (fp_line (start -5.95 -2) (end 5.95 -2) (layer F.CrtYd) (width 0.05))
-    (pad 1 smd rect (at -4.60243 -0.00232) (size 2.18 1.6) (layers F.Cu F.Paste F.Mask)
-      (net 2 GND))
-    (pad 2 smd rect (at 4.60243 0.00232) (size 2.18 1.6) (layers F.Cu F.Paste F.Mask)
-      (net 17 ~RESET))
-  )
   (module KaiBader:CSTCE16M0V53 (layer F.Cu)
-    (at 140.97 117.475)
+    (at 141.605 144.526)
     (descr "CSTCE16M0V53 CERAMIC RESONATOR (CERALOCK) 16 MHZ CHIP TYPE")
     (tags "CSTCE16M0V53 CERAMIC RESONATOR (CERALOCK) 16 MHZ CHIP TYPE")
@@
       (net 10 "Net-(IC1-Pad2)"))
   )
+  (module Buttons_Switches_SMD:SW_SPST_EVQPE1 (layer F.Cu)
+    (at 147.32 146.431)
+    (descr "Light Touch Switch")
+    (attr smd)
+    (fp_text reference SW1 (at -0.9 -2.7) (layer F.SilkS)
+      (effects (font (size 1 1) (thickness 0.15)))
+    )
+    (fp_text value SW_PUSH (at 0 0) (layer F.Fab)
+      (effects (font (size 1 1) (thickness 0.15)))
+    )
+    (fp_line (start -1.4 -0.7) (end 1.4 -0.7) (layer F.SilkS) (width 0.15))
+    (fp_line (start 1.4 -0.7) (end 1.4 0.7) (layer F.SilkS) (width 0.15))
+    (fp_line (start 1.4 0.7) (end -1.4 0.7) (layer F.SilkS) (width 0.15))
+    (fp_line (start -1.4 0.7) (end -1.4 -0.7) (layer F.SilkS) (width 0.15))
+    (fp_line (start -3.95 -2) (end 3.95 -2) (layer F.CrtYd) (width 0.05))
+    (fp_line (start 3.95 -2) (end 3.95 2) (layer F.CrtYd) (width 0.05))
+    (fp_line (start 3.95 2) (end -3.95 2) (layer F.CrtYd) (width 0.05))
+    (fp_line (start -3.95 2) (end -3.95 -2) (layer F.CrtYd) (width 0.05))
+    (fp_line (start 3 -1.75) (end 3 -1.1) (layer F.SilkS) (width 0.15))
+    (fp_line (start 3 1.75) (end 3 1.1) (layer F.SilkS) (width 0.15))
+    (fp_line (start -3 1.1) (end -3 1.75) (layer F.SilkS) (width 0.15))
+    (fp_line (start -3 -1.75) (end -3 -1.1) (layer F.SilkS) (width 0.15))
+    (fp_line (start 3 -1.75) (end -3 -1.75) (layer F.SilkS) (width 0.15))
+    (fp_line (start -3 1.75) (end 3 1.75) (layer F.SilkS) (width 0.15))
+    (pad 2 smd rect (at 2.7 0) (size 2 1.6) (layers F.Cu F.Paste F.Mask)
+      (net 17 ~RESET))
+    (pad 1 smd rect (at -2.7 0) (size 2 1.6) (layers F.Cu F.Paste F.Mask)
+      (net 2 GND))
+  )
   (module KaiBader:AK-S-27_Case (layer F.Cu)
-    (at 127 121.92)
+    (at 127.635 149.225)
     (fp_text reference "" (at 2 0.75) (layer F.Fab) hide
       (effects (font (size 1 1) (thickness 0.15)))
