File: audio_interface.kicad_pcb (KiCad board)
At the start: 2 copper layers, 36 x 14 mm, 26 parts, among them IC1 ATMEGA16U2, P1 USB_A, P2 AVR-ISP, P3 OUT, P4 EAR, Q1 BC849, Q2 BC849, SW1 SW_PUSH, Y1 CSTCE16M0V53MU

Commit message: update
Parts:
- moved P1 123.1 mm to (43.8, 54.0)
- moved R3 120.2 mm to (50.2, 59.7), turned to 0 degrees
- moved R4 119.3 mm to (50.2, 56.5), turned to 0 degrees
- moved Y1 106.2 mm to (114.3, 41.9), turned to 270 degrees
- moved C2 104.5 mm to (121.3, 38.7), turned to 270 degrees
- moved C1 100.7 mm to (119.4, 38.7)
- moved P2 99.2 mm to (118.7, 28.6), turned to 270 degrees
- moved IC1 96.9 mm to (120.7, 44.5), turned to 0 degrees
- moved SW1 94.1 mm to (104.1, 62.9)
- moved R5 92.1 mm to (106.0, 59.7), turned to 180 degrees
- moved R10 89.5 mm to (159.4, 54.0)
- moved C5 88.8 mm to (159.4, 52.1), turned to 0 degrees
- moved C3 86.2 mm to (163.8, 62.2), turned to 180 degrees
- moved C4 86.2 mm to (159.4, 60.3)
- moved R11 85.8 mm to (163.8, 52.1)
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
Commit message: update
Parts:
- moved P1 127.6 mm to (158.8, 109.5)
- moved R3 124.4 mm to (161.5, 115.2), turned to 90 degrees
- moved R4 124.0 mm to (161.5, 111.0), turned to 270 degrees
- moved P2 102.3 mm to (171.0, 116.5), turned to 90 degrees
- moved Y1 88.8 mm to (163.2, 116.0)
- moved C1 88.4 mm to (164.5, 114.8), turned to 180 degrees
- moved IC1 86.2 mm to (169.8, 115.2)
- moved C2 85.9 mm to (164.5, 113.0), turned to 0 degrees
- moved R5 82.6 mm to (172.5, 108.8), turned to 90 degrees
- moved SW1 78.7 mm to (167.5, 109.5)
- moved D1 67.4 mm to (178.8, 117.8), turned to 180 degrees
- moved R1 65.3 mm to (174.0, 117.8), turned to 90 degrees
- moved R11 59.9 mm to (184.0, 108.5)
- moved P4 59.8 mm to (184.0, 111.5)
- moved R6 59.6 mm to (181.0, 117.8), turned to 270 degrees
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